File: PCB and Circuit/Circuit.sch (EAGLE design)
At the start: 3 parts, among them J1 RASPBERRYPI-40-PIN-GPIO_PTH, U1 DS18B20

Commit message: Add files via upload
Connections:
- removed net VCC: J1.GP5
Changed lines of the file:
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@@
 <part name="R1" library="SparkFun-Resistors" library_urn="urn:adsk.eagle:library:532" deviceset="RESISTOR" device="AXIAL-0.3" package3d_urn="urn:adsk.eagle:package:39658/1" value="4K7"/>
 <part name="GND1" library="SparkFun-PowerSymbols" library_urn="urn:adsk.eagle:library:530" deviceset="GND2" device="" value="GND"/>
-<part name="21E12E3" library="supply1" library_urn="urn:adsk.eagle:library:371" deviceset="VCC" device=""/>
 </parts>
 <sheets>
@@
 <instance part="R1" gate="G$1" x="38.1" y="91.44" rot="R270"/>
 <instance part="GND1" gate="G$1" x="35.56" y="10.16"/>
-<instance part="21E12E3" gate="VCC" x="116.84" y="109.22"/>
 </instances>
 <busses>
@@
 </segment>
 </net>
-<net name="VCC" class="0">
-<segment>
-<pinref part="J1" gate="G$1" pin="GP5"/>
-<pinref part="21E12E3" gate="VCC" pin="VCC"/>
-<wire x1="88.9" y1="71.12" x2="116.84" y2="71.12" width="0.1524" layer="91"/>
-<wire x1="116.84" y1="71.12" x2="116.84" y2="106.68" width="0.1524" layer="91"/>
-</segment>
-</net>
